File: usb-power-hub-4/EAGLE/usb-hub-v0.3.brd (EAGLE design)
At the start: 95 x 25 mm, 37 parts, among them U1 RICHTEKRT9715AGBR, U2 RICHTEKRT9715AGBR, U3 RICHTEKRT9715AGBR, U4 RICHTEKRT9715AGBR

Commit message: added missing R5 value
Parts:
- R5: value (none) -> 1k
Changed lines of the file:
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@@
 <attribute name="VALUE" x="13.2715" y="17.145" size="0.4064" layer="27" rot="R90"/>
 </element>
-<element name="R5" library="SparkFun-Resistors" package="0402-RES" value="" x="11.684" y="20.701" smashed="yes">
+<element name="R5" library="SparkFun-Resistors" package="0402-RES" value="1k" x="11.684" y="20.701" smashed="yes">
 <attribute name="NAME" x="12.954" y="20.5105" size="0.4064" layer="25"/>
 <attribute name="VALUE" x="10.6045" y="19.558" size="0.4064" layer="27"/>
